Commit message: fix prefix and set grippers to None

File: prl_ur10e_description/urdf/ur10e_lone_arm.urdf.xacro (robot description, xacro)
@@ -9,9 +9,10 @@
         name:=arm
         ur_type:=ur10e
+        prefix
         parent
         pose
         sensors
-        gripper
-        gripper_pose
+        gripper:=None
+        gripper_pose:=None
         camera:= None
         camera_pose:= None
@@ -34,4 +35,5 @@
         <xacro:ur_robot
             name="ur10"
+            tf_prefix="${prefix}"
             parent="${parent}"
             joint_limits_parameters_file="${joint_limits_parameters_file}"
@@ -59,5 +61,5 @@
         </xacro:if>
         <!-- ROS2 control if real robot -->
-        <xacro:unless value="${gz_sim}">
+        <!-- <xacro:unless value="${gz_sim}">
             <xacro:ur_ros2_control
                 name="ur10"
@@ -76,12 +78,12 @@
                 trajectory_port="${network['trajectory_port']}"s
             />
-        </xacro:unless>
+        </xacro:unless> -->
         <!-- Tool frame -->
-        <link name="${prefix}tool"/>
+        <!-- <link name="${prefix}tool"/>
         <joint name="${prefix}tool_joint" type="fixed">
             <origin xyz="0 0 0" rpy="0 0 ${-pi}"/>
             <parent link="${prefix}robotiq_ft_frame_id"/>
             <child link="${prefix}tool"/>
-        </joint>
+        </joint> -->
     </xacro:macro>
 </robot>
