Commit message: small formatting changes

File: prl_ur10e_description/urdf/ur10e_complete_setup.urdf.xacro (robot description, xacro)
@@ -5,7 +5,7 @@
   <xacro:arg name="real_robot" default="false"/>
   <!-- Setup files -->
-  <xacro:arg name="controller_file" default="$(find ur10e_control)/config/ur10e_controller.yaml"/>  <!-- default="$(find prl_ur5_control)/config/dual_arm_controller.yaml" TODO -->
-  <xacro:property name="setup_file" value="${xacro.load_yaml('$(find ur10e_robot_configuration)/config/standard_setup.yaml')}"/> <!-- TODO -->
-  <!-- ur5 arm -->
+  <xacro:arg name="controller_file" default="$(find prl_ur10e_control)/config/ur10e_controller.yaml"/>
+  <xacro:property name="setup_file" value="${xacro.load_yaml('$(find ur10e_robot_configuration)/config/standard_setup.yaml')}"/>
+  <!-- ur10e arm -->
   <xacro:include filename="$(find prl_ur10e_description)/urdf/ur10e_lone_arm.urdf.xacro"/>
   <!-- fixed camera-->

Commit message: xml parsing error wip fix

File: prl_ur10e_description/urdf/ur10e_complete_setup.urdf.xacro (robot description, xacro)
@@ -9,73 +9,7 @@
   <!-- ur10e arm -->
   <xacro:include filename="$(find prl_ur10e_description)/urdf/ur10e_lone_arm.urdf.xacro"/>
-  <!-- fixed camera-->
-  <!-- <xacro:include filename="$(find prl_ur5_description)/urdf/_fixed_cameras.urdf.xacro"/> -->
   <!-- Global frame -->
   <link name="ur10e_base"/>
-  <!-- Table -->
-  <!-- <material name="Blue">
-    <color rgba="${0/255} ${30/255} ${70/255} 1.0"/>
-  </material>
-  <link name="table_link">
-    <visual>
-      <geometry>
-        <mesh filename="file://$(find prl_ur5_description)/model/vention_table.stl"/>
-      </geometry>
-      <material name="Blue"/>
-    </visual>
-    <collision>
-      <geometry>
-        <mesh filename="file://$(find prl_ur5_description)/model/vention_table.stl"/>
-      </geometry>
-    </collision>
-  </link>
-  <joint name="table_fix" type="fixed">
-    <parent link="prl_ur5_base"/>
-    <child link = "table_link"/>
-    <origin xyz="0.0 0.0 0.0" rpy="0.0 0.0 0.0"/>
-  </joint> -->
-  <!-- Cameras fixtures (if any) -->
-  <!-- <xacro:if value="${setup_file.get('fixed_cameras_file') is not None}">
-    <xacro:fixed_cameras parent="prl_ur5_base" fixed_cameras_file="$(find prl_ur5_robot_configuration)/config/${setup_file['fixed_cameras_file']}" turn_on="true"/>
-  </xacro:if> -->
-  <!-- back wall -->
-  <!-- <link name="backwall_link">
-    <visual>
-      <geometry>
-        <box size="3.5 0.1 2" />
-      </geometry>
-      <material name="grey"><color rgba="0.8 0.8 0.8 0.2"/></material>
-    </visual>
-    <collision>
-      <geometry>
-        <box size="3.5 0.1 2" />
-      </geometry>
-    </collision>
-  </link>
-  <joint name="backwall_fix" type="fixed">
-    <parent link="prl_ur5_base"/>
-    <child link = "backwall_link"/>
-    <origin xyz="0 -1.05 0.25" rpy="0.0 0.0 0.0"/>
-  </joint> -->
-  <!-- left wall -->
-  <!-- <link name="leftwall_link">
-    <visual>
-      <geometry>
-        <box size="0.1 1.95 2" />
-      </geometry>
-      <material name="grey"><color rgba="0.8 0.8 0.8 0.1"/></material>
-    </visual>
-    <collision>
-      <geometry>
-        <box size="0.1 1.95 2" />
-      </geometry>
-    </collision>
-  </link>
-  <joint name="leftwall_fix" type="fixed">
-    <parent link="prl_ur5_base"/>
-    <child link = "leftwall_link"/>
-    <origin xyz="-1.65 0 0.25" rpy="0.0 0.0 0.0"/>
-  </joint> -->
-  <!-- Arm -->
+  <!-- Lone Arm -->
   <xacro:property name="arm" value="${setup_file.get('arm')}"/>
   <xacro:arm parent="prl_ur10e_base"
@@ -87,11 +21,4 @@
                  network = "${arm.get('network')}"
                  />
-  <!-- TO BE added later -->
-  <!--
-                 gripper="${arm.get('gripper')}"
-                 gripper_pose="${arm.get('gripper_pose')}"
-                 camera="${arm.get('camera')}"
-                 camera_pose="${arm.get('camera_pose')}"
-                 -->
   <xacro:if value="$(arg gz_sim)">
     <gazebo>

File: prl_ur10e_description/urdf/ur10e_lone_arm.urdf.xacro (robot description, xacro)
@@ -1,15 +1,8 @@
 <?xml version="1.0"?>
-<robot xmlns:xacro="http://wiki.ros.org/xacro">
-    <!-- ur5 -->
+<robot xmlns:xacro="http://www.ros.org/wiki/xacro">
+    <!-- ur10e -->
     <xacro:include filename="$(find ur_description)/urdf/ur_macro.xacro"/>
     <xacro:include filename="$(find ur_description)/urdf/inc/ur_joint_control.xacro" />
     <xacro:include filename="$(find ur_robot_driver)/urdf/ur.ros2_control.xacro"/>
-<!-- TODO -->
-    <!-- force sensor-->
-    <!-- <xacro:include filename="$(find prl_ur10e_description)/urdf/_force_sensor.urdf.xacro"/> -->
-    <!-- gripper -->
-    <!-- <xacro:include filename="$(find prl_ur10e_description)/urdf/_gripper.urdf.xacro"/> -->
-    <!-- camera -->
-    <!-- <xacro:include filename="$(find prl_ur10e_description)/urdf/_camera_sensor.urdf.xacro"/> -->
     <!-- Macro to define the complete arm -->
     <xacro:macro name="arm" params="
@@ -40,6 +33,5 @@
         <!-- UR10 -->
         <xacro:ur_robot
-            name="${prefix}arm"
-            tf_prefix="${prefix}"
+            name="ur10"
             parent="${parent}"
             joint_limits_parameters_file="${joint_limits_parameters_file}"
@@ -56,5 +48,5 @@
         <!-- ROS2 control if simulation -->
         <xacro:if value="${gz_sim}">
-            <ros2_control name="${prefix}arm" type="system">
+            <ros2_control name="arm" type="system">
                 <hardware>
                     <plugin>gz_ros2_control/GazeboSimSystem</plugin>
@@ -85,10 +77,4 @@
             />
         </xacro:unless>
-        <!-- Force sensor -->
-        <!-- <xacro:force_sensor
-            prefix="${prefix}"
-            parent="tool0"
-            gz_sim="${gz_sim}"
-        /> -->
         <!-- Tool frame -->
         <link name="${prefix}tool"/>
@@ -98,6 +84,4 @@
             <child link="${prefix}tool"/>
         </joint>
-        <!-- Gripper -->
-        <!-- <xacro:gripper gripper="${gripper}" prefix='${prefix}' parent="${prefix}tool" pose="${gripper_pose}" hardware_interface="${hw_interface}" gz_sim="${gz_sim}"/> -->
     </xacro:macro>
 </robot>

Commit message: name fix

File: prl_ur10e_description/urdf/ur10e_complete_setup.urdf.xacro (robot description, xacro)
@@ -6,12 +6,13 @@
   <!-- Setup files -->
   <xacro:arg name="controller_file" default="$(find prl_ur10e_control)/config/ur10e_controller.yaml"/>
-  <xacro:property name="setup_file" value="${xacro.load_yaml('$(find ur10e_robot_configuration)/config/standard_setup.yaml')}"/>
+  <xacro:property name="setup_file" value="${xacro.load_yaml('$(find prl_ur10e_robot_configuration)/config/standard_setup.yaml')}"/>
   <!-- ur10e arm -->
   <xacro:include filename="$(find prl_ur10e_description)/urdf/ur10e_lone_arm.urdf.xacro"/>
   <!-- Global frame -->
-  <link name="ur10e_base"/>
+  <link name="prl_ur10e_base"/>
   <!-- Lone Arm -->
   <xacro:property name="arm" value="${setup_file.get('arm')}"/>
-  <xacro:arm parent="prl_ur10e_base"
+  <xacro:arm prefix="prefix_"
+                 parent="prl_ur10e_base"
                  pose="${arm['arm_pose']}"
                  sensors="false"

Commit message: added dummy table

File: prl_ur10e_description/urdf/ur10e_complete_setup.urdf.xacro (robot description, xacro)
@@ -11,8 +11,30 @@
   <!-- Global frame -->
   <link name="prl_ur10e_base"/>
+  <!-- Base -->
+  <!-- <material name="Blue">
+    <color rgba="${0/255} ${30/255} ${70/255} 1.0"/>
+  </material> -->
+  <link name="table_link">
+    <!-- <visual>
+      <geometry>
+        <mesh filename="file://$(find prl_ur5_description)/model/vention_table.stl"/>
+      </geometry>
+      <material name="Blue"/>
+    </visual> -->
+    <!-- <collision>
+      <geometry>
+        <mesh filename="file://$(find prl_ur5_description)/model/vention_table.stl"/>
+      </geometry>
+    </collision> -->
+  </link>
+  <joint name="table" type="fixed">
+    <parent link="prl_ur10e_base"/>
+    <child link = "table_link"/>
+    <origin xyz="0.0 0.0 0.0" rpy="0.0 0.0 0.0"/>
+  </joint>
   <!-- Lone Arm -->
   <xacro:property name="arm" value="${setup_file.get('arm')}"/>
-  <xacro:arm prefix="prefix_"
-                 parent="prl_ur10e_base"
+  <xacro:arm prefix="ur10_"
+                 parent="table_link"
                  pose="${arm['arm_pose']}"
                  sensors="false"
@@ -34,5 +56,5 @@
     <parent link="base_link" />
     <child link="prl_ur10e_base" />
-    <origin xyz="0 0 0.8" rpy="0 0 0" />
+    <origin xyz="0 0 0.81" rpy="0 0 0" />
   </joint>
 </robot>

File: prl_ur10e_description/urdf/ur10e_lone_arm.urdf.xacro (robot description, xacro)
@@ -34,5 +34,5 @@
         <!-- UR10 -->
         <xacro:ur_robot
-            name="ur10"
+            name="${prefix}arm"
             tf_prefix="${prefix}"
             parent="${parent}"
@@ -63,5 +63,5 @@
         <!-- <xacro:unless value="${gz_sim}">
             <xacro:ur_ros2_control
-                name="ur10"
+                name="${prefix}arm"
                 tf_prefix="${prefix}"
                 kinematics_parameters_file="${kinematics_parameters_file}"

Commit message: adding gripper support

File: prl_ur10e_description/urdf/ur10e_complete_setup.urdf.xacro (robot description, xacro)
@@ -16,4 +16,5 @@
   </material> -->
   <link name="table_link">
+  <!-- TODO -->
     <!-- <visual>
       <geometry>
@@ -39,4 +40,6 @@
                  pose="${arm['arm_pose']}"
                  sensors="false"
+                 gripper="${arm.get('gripper')}"
+                 gripper_pose="${arm.get('gripper_pose')}"
                  gz_sim="$(arg gz_sim)"
                  joint_limits_parameters_file="$(find prl_ur10e_robot_configuration)/config/${arm.get('arm_joint_limits')}"
@@ -44,4 +47,5 @@
                  network = "${arm.get('network')}"
                  />
+  <!-- Gazebosim plugin-->
   <xacro:if value="$(arg gz_sim)">
     <gazebo>

File: prl_ur10e_description/urdf/ur10e_lone_arm.urdf.xacro (robot description, xacro)
@@ -5,4 +5,6 @@
     <xacro:include filename="$(find ur_description)/urdf/inc/ur_joint_control.xacro" />
     <xacro:include filename="$(find ur_robot_driver)/urdf/ur.ros2_control.xacro"/>
+    <!-- gripper -->
+    <xacro:include filename="$(find prl_ur10e_description)/urdf/_gripper.urdf.xacro"/>
     <!-- Macro to define the complete arm -->
     <xacro:macro name="arm" params="
@@ -78,12 +80,14 @@
                 trajectory_port="${network['trajectory_port']}"s
             />
-        </xacro:unless> -->
+        </xacro:unless>  -->
+        <!-- Gripper -->
+        <xacro:gripper gripper="${gripper}" prefix='${prefix}' parent="${prefix}tool" pose="${gripper_pose}" hardware_interface="${hw_interface}" gz_sim="${gz_sim}"/>
         <!-- Tool frame -->
-        <!-- <link name="${prefix}tool"/>
+        <link name="${prefix}tool"/>
         <joint name="${prefix}tool_joint" type="fixed">
             <origin xyz="0 0 0" rpy="0 0 ${-pi}"/>
-            <parent link="${prefix}robotiq_ft_frame_id"/>
+            <parent link="ur10_tool0"/>
             <child link="${prefix}tool"/>
-        </joint> -->
+        </joint>
     </xacro:macro>
 </robot>

Commit message: Added UR stand

File: prl_ur10e_description/urdf/ur10e_complete_setup.urdf.xacro (robot description, xacro)
@@ -12,30 +12,48 @@
   <link name="prl_ur10e_base"/>
   <!-- Base -->
-  <!-- <material name="Blue">
+  <material name="Blue">
     <color rgba="${0/255} ${30/255} ${70/255} 1.0"/>
-  </material> -->
+  </material>
   <link name="table_link">
-  <!-- TODO -->
-    <!-- <visual>
+    <visual>
       <geometry>
-        <mesh filename="file://$(find prl_ur5_description)/model/vention_table.stl"/>
+        <mesh filename="file://$(find prl_ur10e_description)/model/UR10e_stand.stl"/>
       </geometry>
       <material name="Blue"/>
-    </visual> -->
-    <!-- <collision>
+    </visual>
+    <collision>
       <geometry>
-        <mesh filename="file://$(find prl_ur5_description)/model/vention_table.stl"/>
+        <mesh filename="file://$(find prl_ur10e_description)/model/UR10e_stand.stl"/>
       </geometry>
-    </collision> -->
+    </collision>
   </link>
   <joint name="table" type="fixed">
-    <parent link="prl_ur10e_base"/>
+    <parent link="base_link"/>
     <child link = "table_link"/>
     <origin xyz="0.0 0.0 0.0" rpy="0.0 0.0 0.0"/>
   </joint>
+  <!-- left wall -->
+  <!-- <link name="leftwall_link">
+    <visual>
+      <geometry>
+        <box size="0.75 0.75 0.82"/>
+      </geometry>
+      <material name="grey"><color rgba="0.8 0.8 0.8 1"/></material>
+    </visual>
+    <collision>
+      <geometry>
+        <box size="0.75 0.75 0.82"/>
+      </geometry>
+    </collision>
+  </link>
+  <joint name="leftwall_fix" type="fixed">
+    <parent link="prl_ur10e_base"/>
+    <child link = "leftwall_link"/>
+    <origin xyz="0 0 -0.41" rpy="0.0 0.0 0.0"/>
+  </joint> -->
   <!-- Lone Arm -->
   <xacro:property name="arm" value="${setup_file.get('arm')}"/>
   <xacro:arm prefix="ur10_"
-                 parent="table_link"
+                 parent="prl_ur10e_base"
                  pose="${arm['arm_pose']}"
                  sensors="false"
@@ -60,5 +78,5 @@
     <parent link="base_link" />
     <child link="prl_ur10e_base" />
-    <origin xyz="0 0 0.81" rpy="0 0 0" />
+    <origin xyz="0 0 0.82" rpy="0 0 0" />
   </joint>
 </robot>

File: prl_ur10e_description/urdf/ur10e_lone_arm.urdf.xacro (robot description, xacro)
@@ -15,6 +15,6 @@
         pose
         sensors
-        gripper:=None
-        gripper_pose:=None
+        gripper
+        gripper_pose
         camera:= None
         camera_pose:= None

Commit message: cleanup

File: prl_ur10e_description/urdf/ur10e_complete_setup.urdf.xacro (robot description, xacro)
@@ -33,23 +33,4 @@
     <origin xyz="0.0 0.0 0.0" rpy="0.0 0.0 0.0"/>
   </joint>
-  <!-- left wall -->
-  <!-- <link name="leftwall_link">
-    <visual>
-      <geometry>
-        <box size="0.75 0.75 0.82"/>
-      </geometry>
-      <material name="grey"><color rgba="0.8 0.8 0.8 1"/></material>
-    </visual>
-    <collision>
-      <geometry>
-        <box size="0.75 0.75 0.82"/>
-      </geometry>
-    </collision>
-  </link>
-  <joint name="leftwall_fix" type="fixed">
-    <parent link="prl_ur10e_base"/>
-    <child link = "leftwall_link"/>
-    <origin xyz="0 0 -0.41" rpy="0.0 0.0 0.0"/>
-  </joint> -->
   <!-- Lone Arm -->
   <xacro:property name="arm" value="${setup_file.get('arm')}"/>
